Commit message: World

File: src/rover/urdf/rover.urdf (robot description, URDF)
Before this commit: robot rover, 18 links, 17 joints
Links:
- link BackLeftMotor_link: geometry collision mesh filename=file://$(find rover)/meshes/stl/Assem1.006.stl scale=0.00100 0.00100 0.00100; visual mesh filename=file://$(find rover)/meshes/stl/Assem1.006.stl scale=0.00100 0.00100 0.00100
- link BackLeftWheel_link: geometry collision mesh filename=file://$(find rover)/meshes/stl/Assem1.014.stl scale=0.00100 0.00100 0.00100; visual mesh filename=file://$(find rover)/meshes/stl/Assem1.014.stl scale=0.00100 0.00100 0.00100
- link BackRightMotor_link: geometry collision mesh filename=file://$(find rover)/meshes/stl/Assem1.003.stl scale=0.00100 0.00100 0.00100; visual mesh filename=file://$(find rover)/meshes/stl/Assem1.003.stl scale=0.00100 0.00100 0.00100
- link BackRightWheel_link: geometry collision mesh filename=file://$(find rover)/meshes/stl/Assem1.015.stl scale=0.00100 0.00100 0.00100; visual mesh filename=file://$(find rover)/meshes/stl/Assem1.015.stl scale=0.00100 0.00100 0.00100
- link Base_link: geometry collision mesh filename=file://$(find rover)/meshes/stl/Assem1.stl scale=0.00100 0.00100 0.00100; visual mesh filename=file://$(find rover)/meshes/stl/Assem1.stl scale=0.00100 0.00100 0.00100
- link FrontLeftMotor_link: geometry collision mesh filename=file://$(find rover)/meshes/stl/Assem1.009.stl scale=0.00100 0.00100 0.00100; visual mesh filename=file://$(find rover)/meshes/stl/Assem1.009.stl scale=0.00100 0.00100 0.00100
- link FrontLeftWheel_link: geometry collision mesh filename=file://$(find rover)/meshes/stl/Assem1.013.stl scale=0.00100 0.00100 0.00100; visual mesh filename=file://$(find rover)/meshes/stl/Assem1.013.stl scale=0.00100 0.00100 0.00100
- link FrontRightMotor_link: geometry collision mesh filename=file://$(find rover)/meshes/stl/Assem1.012.stl scale=0.00100 0.00100 0.00100; visual mesh filename=file://$(find rover)/meshes/stl/Assem1.012.stl scale=0.00100 0.00100 0.00100
- link FrontRightWheel_link: geometry collision mesh filename=file://$(find rover)/meshes/stl/Assem1.016.stl scale=0.00100 0.00100 0.00100; visual mesh filename=file://$(find rover)/meshes/stl/Assem1.016.stl scale=0.00100 0.00100 0.00100
- link Stand1_link: geometry collision mesh filename=file://$(find rover)/meshes/stl/Assem1.017.stl scale=0.00100 0.00100 0.00100; visual mesh filename=file://$(find rover)/meshes/stl/Assem1.017.stl scale=0.00100 0.00100 0.00100
- link Stand2_link: geometry collision mesh filename=file://$(find rover)/meshes/stl/Assem1.018.stl scale=0.00100 0.00100 0.00100; visual mesh filename=file://$(find rover)/meshes/stl/Assem1.018.stl scale=0.00100 0.00100 0.00100
- link Stand3_link: geometry collision mesh filename=file://$(find rover)/meshes/stl/Assem1.019.stl scale=0.00100 0.00100 0.00100; visual mesh filename=file://$(find rover)/meshes/stl/Assem1.019.stl scale=0.00100 0.00100 0.00100
- link Stand4_link: geometry collision mesh filename=file://$(find rover)/meshes/stl/Assem1.020.stl scale=0.00100 0.00100 0.00100; visual mesh filename=file://$(find rover)/meshes/stl/Assem1.020.stl scale=0.00100 0.00100 0.00100
- link Stand5_link: geometry collision mesh filename=file://$(find rover)/meshes/stl/Assem1.022.stl scale=0.00100 0.00100 0.00100; visual mesh filename=file://$(find rover)/meshes/stl/Assem1.022.stl scale=0.00100 0.00100 0.00100
- link Stand6_link: geometry collision mesh filename=file://$(find rover)/meshes/stl/Assem1.023.stl scale=0.00100 0.00100 0.00100; visual mesh filename=file://$(find rover)/meshes/stl/Assem1.023.stl scale=0.00100 0.00100 0.00100
- link Stand7_link: geometry collision mesh filename=file://$(find rover)/meshes/stl/Assem1.024.stl scale=0.00100 0.00100 0.00100; visual mesh filename=file://$(find rover)/meshes/stl/Assem1.024.stl scale=0.00100 0.00100 0.00100
- link Stand9_link: geometry collision mesh filename=file://$(find rover)/meshes/stl/Assem1.025.stl scale=0.00100 0.00100 0.00100; visual mesh filename=file://$(find rover)/meshes/stl/Assem1.025.stl scale=0.00100 0.00100 0.00100
- link UpperBaseplate_link: geometry collision mesh filename=file://$(find rover)/meshes/stl/Assem1.021.stl scale=0.00100 0.00100 0.00100; visual mesh filename=file://$(find rover)/meshes/stl/Assem1.021.stl scale=0.00100 0.00100 0.00100

Commit message: changes to rsp launch file

File: src/rover/urdf/rover.urdf (robot description, URDF)
Before this commit: robot rover, 18 links, 17 joints
Links:
- added link Camera_link
Joints:
- added joint Camera_link_joint: type fixed, parent Base_link, child Camera_link, origin xyz=0.08613 -0.00106 0.02623 rpy=-1.57060 -1.57057 -1.57099
